Commit message: add robo cruise controller

File: robo_cruiser/urdf/gazebo_mobile_base.xacro (robot description, xacro)
@@ -4,8 +4,8 @@
         <material>Gazebo/Blue</material>
     </gazebo>
-    <gazebo reference="back_right_wheel_link">
+    <gazebo reference="rear_right_wheel_link">
         <material>Gazebo/Grey</material>
     </gazebo>
-    <gazebo reference="back_left_wheel_link">
+    <gazebo reference="rear_left_wheel_link">
         <material>Gazebo/Grey</material>
     </gazebo>
@@ -41,6 +41,6 @@
             <joint_name>base_front_left_steering_wheel_joint</joint_name>
             <joint_name>base_front_right_steering_wheel_joint</joint_name>
-            <joint_name>base_front_right_wheel_joint</joint_name>
-            <joint_name>base_front_left_wheel_joint</joint_name>
+            <joint_name>steering_front_left_wheel_joint</joint_name>
+            <joint_name>steering_front_right_wheel_joint</joint_name>
         </plugin>
     </gazebo>

File: robo_cruiser/urdf/mobile_base.xacro (robot description, xacro)
@@ -99,5 +99,5 @@
         <axis xyz="0 1 0"/>
     </joint> -->
-    <joint name="base_front_right_wheel_joint" type="continuous">
+    <joint name="steering_front_right_wheel_joint" type="continuous">
         <parent link="front_right_steering_wheel_link"/>
         <child link="front_right_wheel_link"/>
@@ -105,5 +105,5 @@
         <axis xyz="0 1 0"/>
     </joint>
-    <joint name="base_front_left_wheel_joint" type="continuous">
+    <joint name="steering_front_left_wheel_joint" type="continuous">
         <parent link="front_left_steering_wheel_link"/>
         <child link="front_left_wheel_link"/>
